Commit message: update

File: Isaacsim_tactile_env/assets/dexmate/vega_1u_gripper_flexitac.urdf (robot description, URDF)
Before this commit: robot vega_1u_gripper_flexitac, 36 links, 35 joints
Links:
- link L_camera_link: geometry collision mesh filename=meshes/wrist_c960_v1/camera_collision.obj; visual mesh filename=meshes/wrist_c960_v1/camera_visual.glb
- link L_gripper_base: geometry collision mesh filename=meshes/wrist_c960_v1/base_collision_0.obj; collision mesh filename=meshes/wrist_c960_v1/base_collision_1.obj
- link L_gripper_l1: geometry collision mesh filename=meshes/pad_66x26_v3/simulation/gripper_l1_metal_collision.o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; collision mesh filename=meshes/pad_66x26_v3/simulation/gripper_l1_tpu_collision.obj
- link L_gripper_l2: geometry collision mesh filename=meshes/pad_66x26_v3/simulation/gripper_l2_metal_collision.o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; collision mesh filename=meshes/pad_66x26_v3/simulation/gripper_l2_tpu_collision.obj
- link R_camera_link: geometry collision mesh filename=meshes/wrist_c960_v1/camera_collision.obj; visual mesh filename=meshes/wrist_c960_v1/camera_visual.glb
- link R_gripper_base: geometry collision mesh filename=meshes/wrist_c960_v1/base_collision_0.obj; collision mesh filename=meshes/wrist_c960_v1/base_collision_1.obj
- link R_gripper_l1: geometry collision mesh filename=meshes/pad_66x26_v3/simulation/gripper_l1_metal_collision.o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; collision mesh filename=meshes/pad_66x26_v3/simulation/gripper_l1_tpu_collision.obj
- link R_gripper_l2: geometry collision mesh filename=meshes/pad_66x26_v3/simulation/gripper_l2_metal_collision.o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; collision mesh filename=meshes/pad_66x26_v3/simulation/gripper_l2_tpu_collision.obj
Joints:
- joint L_camera_joint: origin xyz=0.0002 -0.07459 0.0017504 rpy=-0.087266 0 0 -> xyz=0.000201710843793 -0.0778646601563 -0.00551545286112 rpy=-0.418879020479 -3.67320510335e-06 3.67320510335e-06
- joint R_camera_joint: origin xyz=0.0002 -0.07459 0.0017504 rpy=-0.087266 0 0 -> xyz=0.000201710843793 -0.0778646601563 -0.00551545286112 rpy=-0.418879020479 -3.67320510335e-06 3.67320510335e-06
